File: board/Reference_Keyboard/Reference_Keyboard.kicad_pcb (KiCad board)
At the start: 2 copper layers, 157 x 105 mm, 79 parts, among them J1 Conn_01x03_Pin, J2 USB_C_Receptacle_USB2.0, J3 Conn_01x04_Pin, J4 84953-4, SW1 SW_Push, SW10 SW_Push, SW11 SW_Push, SW12 SW_Push, SW13 SW_Push, SW14 SW_Push, SW15 SW_Push, SW16 SW_Push, SW17 SW_Push, SW18 SW_Push, SW19 SW_Push, SW2 SW_Push, SW20 SW_Push, SW21 SW_Push, SW22 SKQGAFE010, SW23 SKQGAFE010, SW24 RotaryEncoder_Switch, SW3 SW_Push, SW4 SW_Push, SW5 SW_Push, SW6 SW_Push, SW7 SW_Push, SW8 SW_Push, SW9 SW_Push, U1 RP2040, U2 W25Q16JVSSIM, U3 LM1117RS-3.3, Y1 NX3225SA-12MHz-STD-CSR-6

Commit message: Bug fix for the Fn key
Parts:
- added SW23: SKQGAFE010, Button_Switch_SMD:SW_SPST_SKQG_WithStem, F.Cu at (186.7, 116.1)
- SW22: moved to B.Cu
- turned SW22 to 0 degrees
- renumbered SW23 to SW24, SW24 to SW25
Routing:
- net Net-(R5-Pad2): track 8.36 -> 14.8 mm, vias 0 -> 1
- net GND: track 60.2 -> 66.4 mm, vias 1478 -> 1476
