File: board/Reference_Keyboard/Reference_Keyboard.kicad_sch (KiCad schematic)
At the start: 87 parts, among them J1 Conn_01x03_Pin, J2 USB_C_Receptacle_USB2.0, J4 84953-4, SW1 SW_Push, SW10 SW_Push, SW11 SW_Push, SW12 SW_Push, SW13 SW_Push, SW14 SW_Push, SW15 SW_Push, SW16 SW_Push, SW17 SW_Push, SW18 SW_Push, SW19 SW_Push, SW2 SW_Push, SW20 SW_Push, SW21 SW_Push, SW22 SW_Push, SW23 SW_Push, SW24 SW_Push, SW25 SKQGAFE010, SW26 RotaryEncoder_Switch, SW27 SKQGAFE010, SW28 SKQGAFE010, SW3 SW_Push, SW4 SW_Push, SW5 SW_Push, SW6 SW_Push, SW7 SW_Push, SW8 SW_Push, SW9 SW_Push, U1 RP2040, U2 W25Q16JVSSIM, U3 LM1117RS-3.3, Y1 NX3225SA-12MHz-STD-CSR-6

Commit message: Add a current protection circuit
Parts:
- added F1: Polyfuse, Fuse:Fuse_0805_2012Metric, symbol Device:Polyfuse
- D1: value RB161MM-20TR -> RB161MM-20TR
Connections:
- net +5V: now also F1.2; no longer D1.1 (K)
- new net: D1.1 (K), F1.1
Changed lines of the file:
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@@
 	(wire
 		(pts
+			(xy 66.04 129.54) (xy 68.58 129.54)
+		)
+		(stroke
+			(width 0)
+			(type default)
+		)
+	)
+	(wire
+		(pts
 			(xy 90.17 177.8) (xy 100.33 177.8)
 		)
@@
 	(wire
 		(pts
-			(xy 58.42 127) (xy 58.42 129.54)
-		)
-		(stroke
-			(width 0)
-			(type default)
-		)
-	)
-	(wire
-		(pts
 			(xy 99.06 93.98) (xy 110.49 93.98)
 		)
@@
 	(wire
 		(pts
+			(xy 68.58 129.54) (xy 68.58 127)
+		)
+		(stroke
+			(width 0)
+			(type default)
+		)
+	)
+	(wire
+		(pts
 			(xy 165.1 67.31) (xy 165.1 69.85)
 		)
@@
 			)
 		)
-		(property "Value" "RB161MM-20TR "
+		(property "Value" "RB161MM-20TR"
 			(at 49.53 125.73 0)
 			(effects
@@
 	)
 	(symbol
+		(lib_id "Device:Polyfuse")
+		(at 62.23 129.54 90)
+		(unit 1)
+		(exclude_from_sim no)
+		(in_bom yes)
+		(on_board yes)
+		(dnp no)
+		(fields_autoplaced yes)
+		(property "Reference" "F1"
+			(at 62.23 123.19 90)
+			(effects
+				(font
+					(size 1.27 1.27)
+				)
+			)
+		)
+		(property "Value" "Polyfuse"
+			(at 62.23 125.73 90)
+			(effects
+				(font
+					(size 1.27 1.27)
+				)
+			)
+		)
+		(property "Footprint" "Fuse:Fuse_0805_2012Metric"
+			(at 67.31 128.27 0)
+			(effects
+				(font
+					(size 1.27 1.27)
+				)
+				(justify left)
+				(hide yes)
+			)
+		)
+		(property "Datasheet" "~"
+			(at 62.23 129.54 0)
+			(effects
+				(font
+					(size 1.27 1.27)
+				)
+				(hide yes)
+			)
+		)
+		(property "Description" "Resettable fuse, polymeric positive temperature coefficient"
+			(at 62.23 129.54 0)
+			(effects
+				(font
+					(size 1.27 1.27)
+				)
+				(hide yes)
+			)
+		)
+		(pin "1"
+		)
+		(pin "2"
+		)
+		(instances
+			(project ""
+				(path "/488c5a2d-543b-4375-8161-9a6838fbf02d"
+					(reference "F1")
+					(unit 1)
+				)
+			)
+		)
+	)
+	(symbol
 		(lib_id "power:+3.3V")
 		(at 110.49 161.29 0)
@@
 	(symbol
 		(lib_id "power:+5V")
-		(at 58.42 127 0)
+		(at 68.58 127 0)
 		(unit 1)
 		(exclude_from_sim no)
@@
 		(fields_autoplaced yes)
 		(property "Reference" "#PWR028"
-			(at 58.42 130.81 0)
+			(at 68.58 130.81 0)
 			(effects
 				(font
@@
 		)
 		(property "Value" "+5V"
-			(at 58.42 123.4981 0)
+			(at 68.58 123.4981 0)
 			(effects
 				(font
@@
 		)
 		(property "Footprint" ""
-			(at 58.42 127 0)
+			(at 68.58 127 0)
 			(effects
 				(font
@@
 		)
 		(property "Datasheet" ""
-			(at 58.42 127 0)
+			(at 68.58 127 0)
 			(effects
 				(font
@@
 		)
 		(property "Description" ""
-			(at 58.42 127 0)
+			(at 68.58 127 0)
 			(effects
 				(font
