File: board/SSD1306_FFC_Adapter/SSD1306_FFC_Adapter.kicad_pcb (KiCad board)
At the start: 2 copper layers, 22.5 x 31 mm, 10 parts, among them J1 Conn_01x30_Socket, J2 Conn_01x04_Pin

Commit message: Update 3d models
Parts:
- C3: value 1u -> 10u
